File: Stack-chan_GoBottomBase.kicad_pcb (KiCad board)
At the start: 2 copper layers, 23 x 27 mm, 15 parts, among them CN1 CON_USB-C-16p, CN2 CON_GROVE, CN3 CON_USB-C-16p, J1 Conn_01x03, J2 Conn_01x03

Commit message: initial commit
Connections:
- CN2 pad 3: unconnected-(CN2-Pad3) -> +5V
Routing:
- net +5V: track 113.0 -> 117.7 mm
- net /SV2: track 11.4 -> 15.3 mm, vias 0 -> 1
- net Net-(CN1-PadB5): track 30.2 -> 30.8 mm
Changed lines of the file:
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@@
   (net 11 "unconnected-(CN1-PadB7)")
   (net 12 "unconnected-(CN1-PadB8)")
-  (net 13 "unconnected-(CN2-Pad3)")
-  (net 14 "unconnected-(CN3-PadA6)")
-  (net 15 "unconnected-(CN3-PadA7)")
-  (net 16 "unconnected-(CN3-PadA8)")
-  (net 17 "unconnected-(CN3-PadB6)")
-  (net 18 "unconnected-(CN3-PadB7)")
-  (net 19 "unconnected-(CN3-PadB8)")
+  (net 13 "unconnected-(CN3-PadA6)")
+  (net 14 "unconnected-(CN3-PadA7)")
+  (net 15 "unconnected-(CN3-PadA8)")
+  (net 16 "unconnected-(CN3-PadB6)")
+  (net 17 "unconnected-(CN3-PadB7)")
+  (net 18 "unconnected-(CN3-PadB8)")
   (footprint "akita:CON_GROVE_V" (layer "F.Cu")
     (at 5.5 3.25 180)
@@
       (net 4 "/SV2") (pinfunction "2") (pintype "bidirectional") (solder_mask_margin 0.1016))
     (pad "3" thru_hole circle locked (at 1 0 180) (size 1.27 1.27) (drill 0.8) (layers *.Cu *.Mask)
-      (net 13 "unconnected-(CN2-Pad3)") (pinfunction "3") (pintype "bidirectional+no_connect") (solder_mask_margin 0.1016))
+      (net 1 "+5V") (pinfunction "3") (pintype "bidirectional") (solder_mask_margin 0.1016))
     (pad "4" thru_hole circle locked (at 3 0 180) (size 1.27 1.27) (drill 0.8) (layers *.Cu *.Mask)
       (net 2 "GND") (pinfunction "4") (pintype "bidirectional") (solder_mask_margin 0.1016))
@@
       (net 5 "Net-(CN1-PadA5)") (pinfunction "CC1") (pintype "bidirectional"))
     (pad "A6" thru_hole circle (at -0.55 0.675 180) (size 0.8 0.8) (drill 0.5) (layers *.Cu *.Mask)
-      (net 14 "unconnected-(CN3-PadA6)") (pinfunction "DP1") (pintype "bidirectional+no_connect"))
+      (net 13 "unconnected-(CN3-PadA6)") (pinfunction "DP1") (pintype "bidirectional+no_connect"))
     (pad "A7" thru_hole circle (at 0.55 0.675 180) (size 0.8 0.8) (drill 0.5) (layers *.Cu *.Mask)
-      (net 15 "unconnected-(CN3-PadA7)") (pinfunction "DN1") (pintype "bidirectional+no_connect"))
+      (net 14 "unconnected-(CN3-PadA7)") (pinfunction "DN1") (pintype "bidirectional+no_connect"))
     (pad "A8" thru_hole circle (at 1.65 0.675 180) (size 0.8 0.8) (drill 0.5) (layers *.Cu *.Mask)
-      (net 16 "unconnected-(CN3-PadA8)") (pinfunction "SBU1") (pintype "bidirectional+no_connect"))
+      (net 15 "unconnected-(CN3-PadA8)") (pinfunction "SBU1") (pintype "bidirectional+no_connect"))
     (pad "A9" thru_hole circle (at 2.75 0.675 180) (size 0.8 0.8) (drill 0.5) (layers *.Cu *.Mask)
       (net 1 "+5V") (pinfunction "VBUS2") (pintype "bidirectional"))
@@
       (net 9 "Net-(CN1-PadB5)") (pinfunction "CC2") (pintype "bidirectional"))
     (pad "B6" thru_hole circle (at 0.55 -0.675 180) (size 0.8 0.8) (drill 0.5) (layers *.Cu *.Mask)
-      (net 17 "unconnected-(CN3-PadB6)") (pinfunction "DP2") (pintype "bidirectional+no_connect"))
+      (net 16 "unconnected-(CN3-PadB6)") (pinfunction "DP2") (pintype "bidirectional+no_connect"))
     (pad "B7" thru_hole circle (at -0.55 -0.675 180) (size 0.8 0.8) (drill 0.5) (layers *.Cu *.Mask)
-      (net 18 "unconnected-(CN3-PadB7)") (pinfunction "DN2") (pintype "bidirectional+no_connect"))
+      (net 17 "unconnected-(CN3-PadB7)") (pinfunction "DN2") (pintype "bidirectional+no_connect"))
     (pad "B8" thru_hole circle (at -1.65 -0.675 180) (size 0.8 0.8) (drill 0.5) (layers *.Cu *.Mask)
-      (net 19 "unconnected-(CN3-PadB8)") (pinfunction "SBU2") (pintype "bidirectional+no_connect"))
+      (net 18 "unconnected-(CN3-PadB8)") (pinfunction "SBU2") (pintype "bidirectional+no_connect"))
     (pad "B9" thru_hole circle (at -2.75 -0.675 180) (size 0.8 0.8) (drill 0.5) (layers *.Cu *.Mask)
       (net 1 "+5V") (pinfunction "VBUS4") (pintype "bidirectional"))
@@
   (segment (start 14.5 17.5) (end 12.75 19.25) (width 0.4) (layer "F.Cu") (net 1))
   (segment (start 7.18238 17) (end 10.46932 17) (width 1.2) (layer "F.Cu") (net 1))
+  (segment (start 4.5 7.235) (end 5.015 7.75) (width 1.2) (layer "B.Cu") (net 1))
   (segment (start 20 4.345041) (end 21 5.345041) (width 0.4) (layer "B.Cu") (net 1))
   (segment (start 6.765 9.5) (end 8.5 9.5) (width 1.2) (layer "B.Cu") (net 1))
@@
   (segment (start 11.68238 23.31762) (end 11.68238 23.5) (width 0.4) (layer "B.Cu") (net 1))
   (segment (start 20 15.86932) (end 20 16) (width 0.4) (layer "B.Cu") (net 1))
+  (segment (start 4.5 3.25) (end 4.5 7.235) (width 1.2) (layer "B.Cu") (net 1))
   (segment (start 8.75 5.5) (end 4.725 5.5) (width 1.2) (layer "F.Cu") (net 2))
   (segment (start 11.481891 25.799511) (end 9.18238 23.5) (width 0.8) (layer "F.Cu") (net 2))
@@
   (segment (start 8.5 3.25) (end 8.5 6.805) (width 0.2) (layer "B.Cu") (net 3))
   (segment (start 8.5 6.805) (end 7.555 7.75) (width 0.2) (layer "B.Cu") (net 3))
-  (segment (start 6.5 3.25) (end 3.75 6) (width 0.2) (layer "B.Cu") (net 4))
-  (segment (start 3.75 8.430327) (end 6.749673 11.43) (width 0.2) (layer "B.Cu") (net 4))
-  (segment (start 3.75 6) (end 3.75 8.430327) (width 0.2) (layer "B.Cu") (net 4))
-  (segment (start 6.749673 11.43) (end 7.555 11.43) (width 0.2) (layer "B.Cu") (net 4))
+  (segment (start 9.5 9.485) (end 9.5 8.5) (width 0.2) (layer "F.Cu") (net 4))
+  (segment (start 7.555 11.43) (end 9.5 9.485) (width 0.2) (layer "F.Cu") (net 4))
+  (via (at 9.5 8.5) (size 0.6) (drill 0.3) (layers "F.Cu" "B.Cu") (net 4))
+  (segment (start 6.5 2) (end 6.5 3.25) (width 0.2) (layer "B.Cu") (net 4))
+  (segment (start 9 1.5) (end 7 1.5) (width 0.2) (layer "B.Cu") (net 4))
+  (segment (start 10 8) (end 10 2.5) (width 0.2) (layer "B.Cu") (net 4))
+  (segment (start 7 1.5) (end 6.5 2) (width 0.2) (layer "B.Cu") (net 4))
+  (segment (start 9.5 8.5) (end 10 8) (width 0.2) (layer "B.Cu") (net 4))
+  (segment (start 10 2.5) (end 9 1.5) (width 0.2) (layer "B.Cu") (net 4))
   (segment (start 11.806696 11.75) (end 11.825 11.731696) (width 0.2) (layer "F.Cu") (net 5))
   (segment (start 11.825 11.731696) (end 11.825 6) (width 0.2) (layer "F.Cu") (net 5))
@@
   (segment (start 11.825 14.089392) (end 11.207196 14.707196) (width 0.2) (layer "F.Cu") (net 9))
   (via (at 11.207196 14.707196) (size 0.6) (drill 0.3) (layers "F.Cu" "B.Cu") (net 9))
+  (segment (start 16.5 5.075) (end 15.6 4.175) (width 0.2) (layer "B.Cu") (net 9))
   (segment (start 11.92502 15.42502) (end 11.92502 20.73502) (width 0.2) (layer "B.Cu") (net 9))
   (segment (start 11.92502 20.73502) (end 13.19 22) (width 0.2) (layer "B.Cu") (net 9))
   (segment (start 11.207196 14.707196) (end 11.92502 15.42502) (width 0.2) (layer "B.Cu") (net 9))
-  (segment (start 11.207196 11.217824) (end 16.5 5.92502) (width 0.2) (layer "B.Cu") (net 9))
   (segment (start 16.5 19) (end 16.5 20.69) (width 0.2) (layer "B.Cu") (net 9))
   (segment (start 15.6 18.1) (end 16.5 19) (width 0.2) (layer "B.Cu") (net 9))
+  (segment (start 16.5 5.406768) (end 16.5 5.075) (width 0.2) (layer "B.Cu") (net 9))
+  (segment (start 14.906768 7) (end 16.5 5.406768) (width 0.2) (layer "B.Cu") (net 9))
+  (segment (start 11.207196 9.792804) (end 14 7) (width 0.2) (layer "B.Cu") (net 9))
   (segment (start 13.19 22) (end 14.19 22) (width 0.2) (layer "B.Cu") (net 9))
   (segment (start 15.19 22) (end 14.19 22) (width 0.2) (layer "B.Cu") (net 9))
   (segment (start 16.5 20.69) (end 15.19 22) (width 0.2) (layer "B.Cu") (net 9))
+  (segment (start 14 7) (end 14.906768 7) (width 0.2) (layer "B.Cu") (net 9))
   (segment (start 15.6 17.35) (end 15.6 18.1) (width 0.2) (layer "B.Cu") (net 9))
-  (segment (start 11.207196 14.707196) (end 11.207196 11.217824) (width 0.2) (layer "B.Cu") (net 9))
-  (segment (start 16.5 5.92502) (end 16.5 5.075) (width 0.2) (layer "B.Cu") (net 9))
-  (segment (start 16.5 5.075) (end 15.6 4.175) (width 0.2) (layer "B.Cu") (net 9))
+  (segment (start 11.207196 14.707196) (end 11.207196 9.792804) (width 0.2) (layer "B.Cu") (net 9))
   (zone (net 2) (net_name "GND") (layer "F.Cu") (hatch edge 0.508)
     (connect_pads (clearance 0.508))

Commit message: for v1
Parts:
- added SW1: SW_SPDT, akita:SW_SPDT_9x4mm_W2.5mm, B.Cu at (12.0, 14.0)
- moved R2 21.8 mm to (19.5, 26.0)
- moved R1 13.1 mm to (19.5, 23.5)
- moved R4 9.24 mm to (23.3, 26.0), turned to 180 degrees
- moved R3 9.24 mm to (23.3, 23.5), turned to 180 degrees
- moved REF** 4.00 mm to (21.0, 10.0)
- moved J2 3.81 mm to (2.54, 7.62)
- moved CN3 2.77 mm to (20.0, 17.0)
- moved CN1 2.75 mm to (20.0, 3.50)
- moved J1 2.41 mm to (2.54, 10.2)
- moved C2 2.24 mm to (4.99, 16.5)
- moved C4 2.19 mm to (3.81, 14.4)
Connections:
- CN1 pad A4: +5V -> Net-(CN1-PadA4)
- CN1 pad A9: +5V -> Net-(CN1-PadA4)
- CN1 pad B4: +5V -> Net-(CN1-PadA4)
- CN1 pad B9: +5V -> Net-(CN1-PadA4)
- CN3 pad A4: +5V -> Net-(CN1-PadA4)
- CN3 pad A9: +5V -> Net-(CN1-PadA4)
- CN3 pad B4: +5V -> Net-(CN1-PadA4)
- CN3 pad B9: +5V -> Net-(CN1-PadA4)
Routing:
- net Net-(CN1-PadA4): track 0.00 -> 68.6 mm
- net +5V: track 117.7 -> 58.9 mm
- net GND: track 89.6 -> 130.5 mm
- net /SV1: track 4.89 -> 11.3 mm, vias 0 -> 1
- net /SV2: track 15.3 -> 9.75 mm
- net Net-(CN1-PadB5): track 30.8 -> 35.2 mm, vias 1 -> 4
- net Net-(CN1-PadA5): track 40.6 -> 38.8 mm, vias 3 -> 0
Other:
- board size 23 x 27 mm -> 25 x 27 mm
- board text added: "ON"
