File: Stack-chan_GoBottomBase.kicad_sch (KiCad schematic)
At the start: 13 parts, among them CN1 CON_USB-C-16p, CN2 CON_GROVE, CN3 CON_USB-C-16p, J1 Conn_01x03, J2 Conn_01x03

Commit message: for v1
Parts:
- added SW1: SW_SPDT, akita:SW_SPDT_9x4mm_W2.5mm, symbol Switch:SW_SPDT
Connections:
- net +5V: now also SW1.2 (B), SW1.3 (C); no longer CN1.A4 (VBUS1), CN1.A9 (VBUS2), CN1.B4 (VBUS3), CN1.B9 (VBUS4), CN3.A4 (VBUS1), CN3.A9 (VBUS2), CN3.B4 (VBUS3), CN3.B9 (VBUS4)
- new net: CN1.A4 (VBUS1), CN1.A9 (VBUS2), CN1.B4 (VBUS3), CN1.B9 (VBUS4), CN3.A4 (VBUS1), CN3.A9 (VBUS2), CN3.B4 (VBUS3), CN3.B9 (VBUS4), SW1.1 (A)
Changed lines of the file:
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@@
   (junction (at 166.37 62.23) (diameter 0) (color 0 0 0 0)
+  )
+  (junction (at 124.46 43.18) (diameter 0) (color 0 0 0 0)
   )
   (junction (at 93.98 81.28) (diameter 0) (color 0 0 0 0)
@@
     (stroke (width 0) (type default) (color 0 0 0 0))
   )
-  (wire (pts (xy 114.3 45.72) (xy 114.3 58.42))
-    (stroke (width 0) (type default) (color 0 0 0 0))
-  )
   (wire (pts (xy 93.98 78.74) (xy 93.98 81.28))
     (stroke (width 0) (type default) (color 0 0 0 0))
@@
     (stroke (width 0) (type default) (color 0 0 0 0))
   )
+  (wire (pts (xy 114.3 34.29) (xy 124.46 34.29))
+    (stroke (width 0) (type default) (color 0 0 0 0))
+  )
   (wire (pts (xy 72.39 83.82) (xy 93.98 83.82))
     (stroke (width 0) (type default) (color 0 0 0 0))
   )
+  (wire (pts (xy 114.3 40.64) (xy 114.3 34.29))
+    (stroke (width 0) (type default) (color 0 0 0 0))
+  )
+  (wire (pts (xy 128.27 43.18) (xy 128.27 41.91))
+    (stroke (width 0) (type default) (color 0 0 0 0))
+  )
   (wire (pts (xy 147.32 72.39) (xy 154.94 72.39))
     (stroke (width 0) (type default) (color 0 0 0 0))
@@
     (stroke (width 0) (type default) (color 0 0 0 0))
   )
+  (wire (pts (xy 124.46 43.18) (xy 128.27 43.18))
+    (stroke (width 0) (type default) (color 0 0 0 0))
+  )
   (wire (pts (xy 113.03 76.2) (xy 116.84 76.2))
     (stroke (width 0) (type default) (color 0 0 0 0))
@@
     (stroke (width 0) (type default) (color 0 0 0 0))
   )
-  (wire (pts (xy 120.65 58.42) (xy 120.65 54.61))
-    (stroke (width 0) (type default) (color 0 0 0 0))
-  )
   (wire (pts (xy 166.37 62.23) (xy 166.37 60.96))
     (stroke (width 0) (type default) (color 0 0 0 0))
@@
     (stroke (width 0) (type default) (color 0 0 0 0))
   )
+  (wire (pts (xy 124.46 34.29) (xy 124.46 43.18))
+    (stroke (width 0) (type default) (color 0 0 0 0))
+  )
   (wire (pts (xy 102.87 50.8) (xy 93.98 50.8))
     (stroke (width 0) (type default) (color 0 0 0 0))
   )
   (wire (pts (xy 166.37 85.09) (xy 166.37 83.82))
-    (stroke (width 0) (type default) (color 0 0 0 0))
-  )
-  (wire (pts (xy 114.3 58.42) (xy 120.65 58.42))
     (stroke (width 0) (type default) (color 0 0 0 0))
   )
@@
     (pin "2")
   )
-  (symbol (lib_id "power:+5V") (at 120.65 54.61 0) (unit 1)
-    (in_bom yes) (on_board yes) (fields_autoplaced)
-    (property "Reference" "#PWR04" (id 0) (at 120.65 58.42 0)
-      (effects (font (size 1.27 1.27)) hide)
-    )
-    (property "Value" "+5V" (id 1) (at 120.65 51.0055 0))
-    (property "Footprint" "" (id 2) (at 120.65 54.61 0)
-      (effects (font (size 1.27 1.27)) hide)
-    )
-    (property "Datasheet" "" (id 3) (at 120.65 54.61 0)
+  (symbol (lib_id "power:+5V") (at 128.27 41.91 0) (unit 1)
+    (in_bom yes) (on_board yes)
+    (property "Reference" "#PWR04" (id 0) (at 128.27 45.72 0)
+      (effects (font (size 1.27 1.27)) hide)
+    )
+    (property "Value" "+5V" (id 1) (at 128.27 38.3055 0))
+    (property "Footprint" "" (id 2) (at 128.27 41.91 0)
+      (effects (font (size 1.27 1.27)) hide)
+    )
+    (property "Datasheet" "" (id 3) (at 128.27 41.91 0)
       (effects (font (size 1.27 1.27)) hide)
     )
@@
     (pin "1")
   )
+  (symbol (lib_id "Switch:SW_SPDT") (at 119.38 43.18 180) (unit 1)
+    (in_bom yes) (on_board yes) (fields_autoplaced)
+    (property "Reference" "SW1" (id 0) (at 119.38 36.2925 0))
+    (property "Value" "SW_SPDT" (id 1) (at 119.38 39.0676 0))
+    (property "Footprint" "akita:SW_SPDT_9x4mm_W2.5mm" (id 2) (at 119.38 43.18 0)
+      (effects (font (size 1.27 1.27)) hide)
+    )
+    (property "Datasheet" "~" (id 3) (at 119.38 43.18 0)
+      (effects (font (size 1.27 1.27)) hide)
+    )
+    (pin "1")
+    (pin "2")
+    (pin "3")
+  )
   (sheet_instances
     (path "/" (page "1"))
@@
       (reference "R4") (unit 1) (value "5.1k") (footprint "Resistor_THT:R_Axial_DIN0204_L3.6mm_D1.6mm_P7.62mm_Horizontal")
     )
-  )
+    (path "/f9c966ae-23e4-43cd-95e1-ebb675260935"
+      (reference "SW1") (unit 1) (value "SW_SPDT") (footprint "akita:SW_SPDT_9x4mm_W2.5mm")
+    )
+  )
